File: pcb/ai_orb-8.brd (EAGLE design)
At the start: 44.5 x 44.5 mm, 30 parts

Commit message: updating
Parts:
- removed LED10, LED12, LED14, LED16, LED2, LED4, LED6, LED8: LED-WS2812B-SM, Ai_LED:LED-WS2812B-SM
- added +', -', DI', DO': 1X01-PETAL, Ai_Connectors:1X01-PETAL
- added LOGO1: AI-LOGOXS, Ai_Miscellany:AI-LOGO-XS
- moved DO 28.1 mm to (11.2, 5.69)
- moved + 28.0 mm to (5.66, 33.2)
- moved DI 0.10 mm to (33.2, 38.8)
- moved - 0.07 mm to (26.1, 2.77)
Connections:
- removed net N$11: LED10.2, LED11.4
- removed net N$12: LED11.2, LED12.4
- removed net N$15: LED14.2, LED15.4
- removed net N$16: LED15.2, LED16.4
- removed net N$3: DI.1, R1.2
- removed net N$5: LED4.2, LED5.4
- removed net N$7: LED6.2, LED7.4
- removed net N$8: LED7.2, LED8.4
- net DO: now also DO'.1, LED15.2; no longer LED16.2
- net GND: now also -'.1; no longer LED10.3, LED12.3, LED14.3, LED16.3, LED2.3, LED4.3, LED6.3, LED8.3
- net N$1: now also LED3.4; no longer LED2.4
- net N$10: now also LED11.4; no longer LED10.4
- net N$13: now also LED11.2; no longer LED12.2
- net N$14: now also LED15.4; no longer LED14.4
- net N$2: now also DI'.1, DI.1, R1.2; no longer LED2.2, LED3.4
- net N$4: now also LED5.4; no longer LED4.4
- net N$6: now also LED7.4; no longer LED6.4
- net N$9: now also LED7.2; no longer LED8.2
- net VCC: now also +'.1; no longer LED10.1, LED12.1, LED14.1, LED16.1, LED2.1, LED4.1, LED6.1, LED8.1
Routing:
- net DO: track 9.32 -> 35.5 mm
- net N$3: track 15.3 -> 0.00 mm
- net N$8: track 12.5 -> 0.00 mm, vias 2 -> 0
- net N$15: track 12.5 -> 0.00 mm, vias 2 -> 0
- net N$12: track 12.5 -> 0.00 mm, vias 2 -> 0
- net N$11: track 12.5 -> 0.00 mm, vias 2 -> 0
- net N$16: track 12.5 -> 0.00 mm, vias 2 -> 0
- net N$5: track 12.5 -> 0.00 mm, vias 2 -> 0
- net N$7: track 12.5 -> 0.00 mm, vias 2 -> 0
- net N$6: track 12.5 -> 23.2 mm
- net N$2: track 12.5 -> 22.2 mm, vias 2 -> 1
- net N$4: track 12.5 -> 22.1 mm
- net N$1: track 12.5 -> 22.0 mm, vias 3 -> 2
- net N$10: track 12.4 -> 19.6 mm
- net N$9: track 12.5 -> 19.6 mm
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Other:
- board text added: "ORB-8"
- board text removed: "ORB-16"

Commit message: updating files
Routing:
- net N$2: track 22.2 -> 23.2 mm
Other:
- board text added: "v1.1"
- board text removed: "v1.0"
Changed lines of the file:
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@@
 <setting verticaltext="up"/>
 </settings>
-<grid distance="5" unitdist="mil" unit="mil" style="lines" multiple="1" display="yes" altdistance="0.025" altunitdist="inch" altunit="inch"/>
+<grid distance="1" unitdist="mil" unit="mil" style="lines" multiple="1" display="yes" altdistance="0.025" altunitdist="inch" altunit="inch"/>
 <layers>
 <layer number="1" name="Top" color="4" fill="1" visible="yes" active="yes"/>
@@
 <text x="4.826" y="15.367" size="1.016" layer="22" font="vector" ratio="10" rot="SMR235">ORB-8</text>
 <text x="27.432" y="5.334" size="1.016" layer="22" font="vector" ratio="10" rot="SMR0">Pasadena, CA</text>
-<text x="23.622" y="0.254" size="0.762" layer="22" font="vector" ratio="10" rot="MR0">v1.0</text>
+<text x="23.622" y="0.254" size="0.762" layer="22" font="vector" ratio="10" rot="MR0">v1.1</text>
 </plain>
 <attributes>
@@
 <wire x1="2.921" y1="21.7678" x2="2.92361875" y2="26.061146875" width="0.4064" layer="1"/>
 <wire x1="2.92361875" y1="26.061146875" x2="3.683" y2="29.718" width="0.4064" layer="1"/>
-<wire x1="20.025" y1="42.875" x2="22.1742" y2="41.529" width="0.4064" layer="1"/>
-<via x="22.1742" y="41.529" extent="1-16" drill="0.508"/>
+<via x="22.0726" y="42.1132" extent="1-16" drill="0.508"/>
 <wire x1="18.7452" y1="41.529" x2="16.637" y2="41.0718" width="0.4064" layer="16"/>
 <via x="16.637" y="41.0718" extent="1-16" drill="0.508"/>
 <wire x1="16.637" y1="41.0718" x2="11.308990625" y2="38.575859375" width="0.4064" layer="1"/>
-<wire x1="22.1742" y1="41.529" x2="26.061146875" y2="41.526378125" width="0.4064" layer="1"/>
+<wire x1="22.0726" y1="42.1132" x2="23.5966" y2="41.5544" width="0.4064" layer="1"/>
+<wire x1="23.5966" y1="41.5544" x2="26.061146875" y2="41.526378125" width="0.4064" layer="1"/>
 <wire x1="39.3488125" y1="31.802534375" x2="38.575859375" y2="33.14100625" width="0.4064" layer="1"/>
 <wire x1="42.875" y1="24.425" x2="41.3004" y2="22.225" width="0.4064" layer="1"/>
@@
 <wire x1="8.8392" y1="8.3566" x2="5.8741375" y2="11.308990625" width="0.4064" layer="1"/>
 <wire x1="5.8741375" y1="11.308990625" x2="1.575" y2="20.025" width="0.4064" layer="1"/>
-<wire x1="18.7452" y1="41.529" x2="22.1742" y2="41.529" width="0.4064" layer="16"/>
+<wire x1="18.7452" y1="41.529" x2="22.0726" y2="42.1132" width="0.4064" layer="16"/>
 <wire x1="35.262734375" y1="38.374003125" x2="35.1028" y2="36.6522" width="0.4064" layer="1"/>
 <wire x1="35.1028" y1="36.6522" x2="38.575859375" y2="33.14100625" width="0.4064" layer="1"/>
 <wire x1="38.575859375" y1="33.14100625" x2="39.3488125" y2="31.802534375" width="0.4064" layer="16"/>
 <via x="39.3488125" y="31.802534375" extent="1-16" drill="0.508"/>
-<wire x1="26.061146875" y1="41.526378125" x2="26.0604" y2="38.9128" width="0.4064" layer="1"/>
+<wire x1="26.061146875" y1="41.526378125" x2="25.8826" y2="41.3512" width="0.4064" layer="1"/>
+<wire x1="25.8826" y1="41.3512" x2="25.8826" y2="39.116" width="0.4064" layer="1"/>
+<wire x1="25.8826" y1="39.116" x2="26.0604" y2="38.9128" width="0.4064" layer="1"/>
 <wire x1="26.0604" y1="38.9128" x2="27.813" y2="38.6842" width="0.4064" layer="1"/>
 <wire x1="27.813" y1="38.6842" x2="30.6832" y2="37.3634" width="0.4064" layer="1"/>
@@
 <via x="22.1996" y="3.175" extent="1-16" drill="0.508"/>
 <wire x1="22.1996" y1="3.175" x2="18.90209375" y2="3.183065625" width="0.4064" layer="1"/>
-</signal>
-<signal name="GND" airwireshidden="yes">
+<wire x1="20.025" y1="42.875" x2="22.0726" y2="42.1132" width="0.4064" layer="1"/>
+</signal>
+<signal name="GND">
 <contactref element="LED7" pad="3"/>
 <contactref element="LED1" pad="3"/>
@@
 <contactref element="-" pad="1"/>
 <contactref element="-'" pad="1"/>
-<wire x1="24.425" y1="39.675" x2="11.450003125" y2="36.1112625" width="0" layer="19" extent="1-1"/>
-<wire x1="26.31365" y1="42.80161875" x2="24.425" y2="39.675" width="0" layer="19" extent="1-1"/>
+<via x="26.8986" y="39.751" extent="1-16" drill="0.508"/>
+<via x="37.3126" y="30.226" extent="1-16" drill="0.508"/>
+<via x="36.703" y="13.589" extent="1-16" drill="0.508"/>
+<via x="3.0988" y="13.4366" extent="1-16" drill="0.508"/>
+<via x="22.1488" y="40.4876" extent="1-16" drill="0.508"/>
 </signal>
 <signal name="N$1">
@@
 <contactref element="R1" pad="2"/>
 <contactref element="DI" pad="1"/>
-<wire x1="18.3899625" y1="41.5266" x2="18.1102" y2="40.4114" width="0.4064" layer="1"/>
-<wire x1="18.1102" y1="40.4114" x2="18.3896" y2="38.7604" width="0.4064" layer="1"/>
-<wire x1="18.3896" y1="38.7604" x2="18.6944" y2="38.481" width="0.4064" layer="16"/>
+<wire x1="17.7546" y1="39.3954" x2="18.5928" y2="38.4556" width="0.4064" layer="16"/>
 <wire x1="22.4536" y1="38.735" x2="27.5336" y2="38.0238" width="0.4064" layer="16"/>
-<wire x1="27.5336" y1="38.0238" x2="28.829" y2="37.4142" width="0.4064" layer="16"/>
-<wire x1="28.829" y1="37.4142" x2="32.5628" y2="38.735" width="0.4064" layer="16"/>
-<wire x1="32.5628" y1="38.735" x2="33.2232" y2="38.7604" width="0.4064" layer="16"/>
-<via x="18.3896" y="38.7604" extent="1-16" drill="0.508"/>
-<wire x1="22.4536" y1="38.735" x2="18.6944" y2="38.481" width="0.4064" layer="16"/>
+<wire x1="27.5336" y1="38.0238" x2="29.9974" y2="36.8554" width="0.4064" layer="16"/>
+<wire x1="29.9974" y1="36.8554" x2="31.3182" y2="36.9062" width="0.4064" layer="16"/>
+<wire x1="31.3182" y1="36.9062" x2="33.2232" y2="38.7604" width="0.4064" layer="16"/>
+<via x="17.7546" y="39.3954" extent="1-16" drill="0.508"/>
+<wire x1="22.4536" y1="38.735" x2="18.5928" y2="38.4556" width="0.4064" layer="16"/>
 <contactref element="DI'" pad="1"/>
 <wire x1="29.718" y1="40.767" x2="33.2232" y2="38.7604" width="0.4064" layer="1"/>
+<wire x1="18.3899625" y1="41.5266" x2="17.7546" y2="39.3954" width="0.4064" layer="1"/>
 </signal>
 </signals>
