File: pcb/ai_orb-8.sch (EAGLE design)
At the start: 30 parts

Commit message: updating
Parts:
- removed LED10, LED12, LED14, LED16, LED2, LED4, LED6, LED8: LED-WS2812B-SM, Ai_LED:LED-WS2812B-SM
- added +', -', DI', DO': 1X01-PETAL, Ai_Connectors:1X01-PETAL
- added LOGO1: AI-LOGOXS, Ai_Miscellany:AI-LOGOXS
Connections:
- removed net N$11: LED10.DO, LED11.DI
- removed net N$12: LED11.DO, LED12.DI
- removed net N$15: LED14.DO, LED15.DI
- removed net N$16: LED15.DO, LED16.DI
- removed net N$3: DI.1, R1.2
- removed net N$5: LED4.DO, LED5.DI
- removed net N$7: LED6.DO, LED7.DI
- removed net N$8: LED7.DO, LED8.DI
- net DO: now also DO'.1, LED15.DO; no longer LED16.DO
- net GND: now also -'.1; no longer LED10.VSS, LED12.VSS, LED14.VSS, LED16.VSS, LED2.VSS, LED4.VSS, LED6.VSS, LED8.VSS
- net N$1: now also LED3.DI; no longer LED2.DI
- net N$10: now also LED11.DI; no longer LED10.DI
- net N$13: now also LED11.DO; no longer LED12.DO
- net N$14: now also LED15.DI; no longer LED14.DI
- net N$2: now also DI'.1, DI.1, R1.2; no longer LED2.DO, LED3.DI
- net N$4: now also LED5.DI; no longer LED4.DI
- net N$6: now also LED7.DI; no longer LED6.DI
- net N$9: now also LED7.DO; no longer LED8.DO
- net VCC: now also +'.1; no longer LED10.VDD, LED12.VDD, LED14.VDD, LED16.VDD, LED2.VDD, LED4.VDD, LED6.VDD, LED8.VDD
Other:
- moved on the sheet: +, -, DI, DO, LED11, LED13, LED15, LED3, LED5, LED7, LED9, R1
